File: Sudden_XCVR_IF_Module.brd (EAGLE design)
At the start: 160 x 100 mm, 25 parts

Commit message: Lots of changes.
Recreated the IF Schema and a new board to look like the photo

On branch master
Changes to be committed:
       modified:   Receiver RF Amplifier Stage.b#1
       modified:   Receiver RF Amplifier Stage.b#2
       modified:   Receiver RF Amplifier Stage.b#3
       modified:   Receiver RF Amplifier Stage.b#4
       modified:   Receiver RF Amplifier Stage.b#5
       modified:   Receiver RF Amplifier Stage.b#6
       modified:   Receiver RF Amplifier Stage.b#7
       modified:   Receiver RF Amplifier Stage.b#8
       modified:   Receiver RF Amplifier Stage.b#9
       modified:   Receiver RF Amplifier Stage.brd
       modified:   Receiver RF Amplifier Stage.s#1
       modified:   Receiver RF Amplifier Stage.s#2
       modified:   Receiver RF Amplifier Stage.s#3
       modified:   Receiver RF Amplifier Stage.s#4
       modified:   Receiver RF Amplifier Stage.s#5
       modified:   Receiver RF Amplifier Stage.s#6
       modified:   Receiver RF Amplifier Stage.s#7
       modified:   Receiver RF Amplifier Stage.s#8
       modified:   Receiver RF Amplifier Stage.s#9
       modified:   Receiver RF Amplifier Stage.sch
       modified:   Sudden_XCVR_IF_Module.b#1
       modified:   Sudden_XCVR_IF_Module.b#2
       modified:   Sudden_XCVR_IF_Module.b#3
       modified:   Sudden_XCVR_IF_Module.b#4
       modified:   Sudden_XCVR_IF_Module.b#5
       modified:   Sudden_XCVR_IF_Module.b#6
       modified:   Sudden_XCVR_IF_Module.b#7
       modified:   Sudden_XCVR_IF_Module.brd
       new file:   Sudden_XCVR_IF_Module_Schematic_like_board_layout.b#1
       new file:   Sudden_XCVR_IF_Module_Schematic_like_board_layout.b#2
       new file:   Sudden_XCVR_IF_Module_Schematic_like_board_layout.b#3
       new file:   Sudden_XCVR_IF_Module_Schematic_like_board_layout.brd
       new file:   Sudden_XCVR_IF_Module_Schematic_like_board_layout.s#1
       new file:   Sudden_XCVR_IF_Module_Schematic_like_board_layout.s#2
       new file:   Sudden_XCVR_IF_Module_Schematic_like_boa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
Parts:
- moved C9 200.7 mm to (-48.3, 58.4), turned to 0 degrees
- moved C10 197.7 mm to (-58.4, 58.4), turned to 0 degrees
- moved C8 189.4 mm to (-38.1, 58.4), turned to 0 degrees
- moved H4 189.4 mm to (-38.1, 24.1)
- moved L2 187.9 mm to (-61.0, 66.0), turned to 0 degrees
- moved H3 183.9 mm to (-27.9, 24.1)
- moved C7 151.8 mm to (-27.9, 58.4), turned to 0 degrees
- moved C12 144.6 mm to (-27.9, 33.0), turned to 0 degrees
- moved C6 133.7 mm to (-17.8, 58.4)
- moved IC2 132.9 mm to (26.7, 121.9), turned to 180 degrees
- moved P+1 127.9 mm to (-16.5, 72.4)
- moved Q1 127.6 mm to (54.6, 139.7), turned to 0 degrees
- moved L5 114.1 mm to (36.8, 124.5), turned to 90 degrees
- moved IC1 100.0 mm to (81.3, 121.9), turned to 180 degrees
- moved H1 97.1 mm to (-57.1, 6.35)
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Routing:
- net N$9: track 68.2 -> 0.00 mm
- net N$1: track 58.0 -> 0.00 mm
- net +5V: track 45.6 -> 0.00 mm
- net N$16: track 35.4 -> 0.00 mm
- net N$17: track 34.9 -> 0.00 mm, vias 1 -> 0
- net N$4: track 17.8 -> 0.00 mm
- net N$7: track 17.3 -> 0.00 mm
- net N$3: track 17.3 -> 0.00 mm
- net N$2: track 16.7 -> 0.00 mm
- net N$14: track 16.0 -> 0.00 mm
- net N$20: track 16.0 -> 0.00 mm
- net N$15: track 16.0 -> 0.00 mm
- net N$19: track 14.8 -> 0.00 mm
- net N$6: track 13.5 -> 0.00 mm
- net N$5: track 13.5 -> 0.00 mm
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- removed copper zone on layer 1, net GND
Other:
- board size 160 x 100 mm -> 109.2 x 150.8 mm
