File: Sudden_XCVF_Driver_Stage.brd (EAGLE design)
At the start: 63.5 x 61.9 mm, 14 parts, among them Q1 2N2222

Commit message: On branch master Changes to be committed:        modified:   Sudden_XCVF_Driver_Stage.b#1        modified:   Sudden_XCVF_Driver_Stage.b#2        modified:   Sudden_XCVF_Driver_Stage.b#3        modified:   Sudden_XCVF_Driver_Stage.b#4        modified:   Sudden_XCVF_Driver_Stage.b#5        new file:   Sudden_XCVF_Driver_Stage.b#6        new file:   Sudden_XCVF_Driver_Stage.b#7        modified:   Sudden_XCVF_Driver_Stage.brd        modified:   Sudden_XCVF_Driver_Stage.s#1        modified:   Sudden_XCVF_Driver_Stage.s#2        modified:   Sudden_XCVF_Driver_Stage.s#4        new file:   Sudden_XCVF_Driver_Stage.s#5        modified:   Sudden_XCVF_Driver_Stage.sch        modified:   eagle.epf
Parts:
- removed R8: 50R, jim_muppet_parts:RESITOR-MUPPET
- added H2: AC Signal Out, jim_muppet_parts:PAD-SQUARE
- Q1: value 2N2222 -> 2N2219A
Connections:
- net GND: no longer R8.P$2
- net N$3: now also H2.PAD; no longer R8.P$1
Routing:
- net N$3: track 10.6 -> 12.7 mm
