File: Sudden_XCVR_Mic_Amp.brd (EAGLE design)
At the start: 81.3 x 63.2 mm, 14 parts, among them T1 2N3904

Commit message: Added Mic Amp
Added Mic Amp, not sure this will conflict with previous commit

On branch master
Changes to be committed:
       modified:   Sudden_XCVR_Mic_Amp.b#1
       modified:   Sudden_XCVR_Mic_Amp.b#2
       modified:   Sudden_XCVR_Mic_Amp.b#3
       new file:   Sudden_XCVR_Mic_Amp.b#4
       modified:   Sudden_XCVR_Mic_Amp.brd
       modified:   Sudden_XCVR_Mic_Amp.s#1
       modified:   Sudden_XCVR_Mic_Amp.s#2
       new file:   Sudden_XCVR_Mic_Amp.s#3
       modified:   Sudden_XCVR_Mic_Amp.sch
Parts:
- moved T1 3.81 mm to (40.6, 31.8)
- moved R4 2.84 mm to (44.5, 16.5)
- moved C1 2.54 mm to (12.7, 41.9)
- moved C3 1.27 mm to (14.0, 30.5)
Routing:
- net N$4: track 0.00 -> 39.9 mm
- net N$2: track 0.00 -> 26.1 mm
- net N$1: track 0.00 -> 24.1 mm
- net N$8: track 0.00 -> 13.5 mm
- net N$5: track 0.00 -> 12.5 mm
- net +12V: track 0.00 -> 11.2 mm
- net N$6: track 0.00 -> 10.9 mm
- net N$7: track 0.00 -> 10.2 mm
- net N$3: track 0.00 -> 8.92 mm
Changed lines of the file:
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@@
 </variantdefs>
 <classes>
-<class number="0" name="default" width="0" drill="0">
+<class number="0" name="default" width="0.9398" drill="0">
+<clearance class="0" value="0.9398"/>
 </class>
 </classes>
@@
 </autorouter>
 <elements>
-<element name="C1" library="jim_muppet_parts" package="CAP-POLARIZED" package3d_urn="urn:adsk.eagle:package:37415/1" value="100uF" x="12.7" y="44.45" smashed="yes" rot="R90">
-<attribute name="NAME" x="9.271" y="44.45" size="0.6096" layer="25" font="vector" ratio="20" rot="R90" align="bottom-center"/>
-<attribute name="PROD_ID" value="CAP-08439" x="34.29" y="82.55" size="1.778" layer="27" rot="R90" display="off"/>
-<attribute name="VALUE" x="16.129" y="44.45" size="0.6096" layer="27" font="vector" ratio="20" rot="R90" align="top-center"/>
+<element name="C1" library="jim_muppet_parts" package="CAP-POLARIZED" package3d_urn="urn:adsk.eagle:package:37415/1" value="100uF" x="12.7" y="41.91" smashed="yes" rot="R90">
+<attribute name="NAME" x="9.271" y="41.91" size="0.6096" layer="25" font="vector" ratio="20" rot="R90" align="bottom-center"/>
+<attribute name="PROD_ID" value="CAP-08439" x="34.29" y="80.01" size="1.778" layer="27" rot="R90" display="off"/>
+<attribute name="VALUE" x="16.129" y="41.91" size="0.6096" layer="27" font="vector" ratio="20" rot="R90" align="top-center"/>
 </element>
 <element name="C2" library="jim_muppet_parts" package="CAP-POLARIZED" package3d_urn="urn:adsk.eagle:package:37415/1" value="470uF" x="60.96" y="15.24" smashed="yes" rot="R90">
@@
 <attribute name="VALUE" x="64.389" y="15.24" size="0.6096" layer="27" font="vector" ratio="20" rot="R90" align="top-center"/>
 </element>
-<element name="C3" library="jim_muppet_parts" package="CAP-MEDIUM-MUPPET" value="10uF" x="13.97" y="29.21" smashed="yes" rot="R270">
-<attribute name="NAME" x="15.875" y="32.893" size="1.27" layer="25" font="vector" rot="R270"/>
-<attribute name="PROD_ID" value="JIM-CAP Large SMT" x="-34.29" y="11.43" size="1.778" layer="27" rot="R270" display="off"/>
-<attribute name="VALUE" x="10.795" y="33.147" size="1.27" layer="27" font="vector" rot="R270"/>
+<element name="C3" library="jim_muppet_parts" package="CAP-MEDIUM-MUPPET" value="10uF" x="13.97" y="30.48" smashed="yes" rot="R270">
+<attribute name="NAME" x="15.875" y="34.163" size="1.27" layer="25" font="vector" rot="R270"/>
+<attribute name="PROD_ID" value="JIM-CAP Large SMT" x="-34.29" y="12.7" size="1.778" layer="27" rot="R270" display="off"/>
+<attribute name="VALUE" x="10.795" y="34.417" size="1.27" layer="27" font="vector" rot="R270"/>
 </element>
 <element name="C4" library="jim_muppet_parts" package="CAP-MEDIUM-MUPPET" value="2.2uF" x="55.88" y="46.99" smashed="yes">
@@
 <attribute name="VALUE" x="27.432" y="40.513" size="1.27" layer="27" rot="R90"/>
 </element>
-<element name="R4" library="jim_muppet_parts" package="RESITOR-MUPPET" value="1K" x="45.72" y="19.05" smashed="yes" rot="R90">
-<attribute name="NAME" x="43.688" y="15.24" size="1.27" layer="25" rot="R90"/>
-<attribute name="PROD_ID" value="MUP-RES" x="86.36" y="36.83" size="1.778" layer="27" rot="R90" display="off"/>
-<attribute name="VALUE" x="49.022" y="15.113" size="1.27" layer="27" rot="R90"/>
+<element name="R4" library="jim_muppet_parts" package="RESITOR-MUPPET" value="1K" x="44.45" y="16.51" smashed="yes" rot="R90">
+<attribute name="NAME" x="42.418" y="12.7" size="1.27" layer="25" rot="R90"/>
+<attribute name="PROD_ID" value="MUP-RES" x="85.09" y="34.29" size="1.778" layer="27" rot="R90" display="off"/>
+<attribute name="VALUE" x="47.752" y="12.573" size="1.27" layer="27" rot="R90"/>
 </element>
 <element name="R5" library="jim_muppet_parts" package="RESITOR-MUPPET" value="2.2K" x="41.91" y="53.34" smashed="yes" rot="R180">
@@
 <attribute name="VALUE" x="29.337" y="56.642" size="1.27" layer="27" rot="R180"/>
 </element>
-<element name="T1" library="jim_muppet_parts" package="TO92" package3d_urn="urn:adsk.eagle:package:29893/2" value="2N3904" x="40.64" y="35.56" smashed="yes" rot="R90">
-<attribute name="NAME" x="38.735" y="40.513" size="1.27" layer="25" ratio="10" rot="R90"/>
-<attribute name="VALUE" x="39.37" y="25.908" size="1.27" layer="27" ratio="10" rot="R90"/>
+<element name="T1" library="jim_muppet_parts" package="TO92" package3d_urn="urn:adsk.eagle:package:29893/2" value="2N3904" x="40.64" y="31.75" smashed="yes" rot="R90">
+<attribute name="NAME" x="38.735" y="36.703" size="1.27" layer="25" ratio="10" rot="R90"/>
+<attribute name="VALUE" x="39.37" y="22.098" size="1.27" layer="27" ratio="10" rot="R90"/>
 </element>
 <element name="H1" library="jim_muppet_parts" package="PAD-SQUARE" package3d_urn="urn:adsk.eagle:package:14295/1" value="Mic Signal Out" x="71.12" y="35.56" smashed="yes"/>
@@
 <contactref element="R5" pad="P$1"/>
 <contactref element="C4" pad="1"/>
-<wire x1="44.704" y1="53.34" x2="52.871" y2="46.99" width="0" layer="19" extent="1-1"/>
-<wire x1="44.831" y1="41.275" x2="44.704" y2="53.34" width="0" layer="19" extent="1-1"/>
+<wire x1="44.704" y1="53.34" x2="44.704" y2="46.99" width="0.9398" layer="1"/>
+<wire x1="44.704" y1="46.99" x2="44.704" y2="37.592" width="0.9398" layer="1"/>
+<wire x1="44.704" y1="37.592" x2="44.831" y2="37.465" width="0.9398" layer="1"/>
+<wire x1="52.871" y1="46.99" x2="44.704" y2="46.99" width="0.9398" layer="1"/>
 </signal>
 <signal name="N$2">
@@
 <contactref element="R4" pad="P$2"/>
 <contactref element="C2" pad="1"/>
-<wire x1="60.96" y1="17.887" x2="45.72" y2="21.844" width="0" layer="19" extent="1-1"/>
-<wire x1="44.831" y1="30.861" x2="60.96" y2="17.887" width="0" layer="19" extent="1-1"/>
+<wire x1="44.831" y1="27.051" x2="44.831" y2="22.86" width="0.9398" layer="1"/>
+<wire x1="44.831" y1="22.86" x2="44.831" y2="19.685" width="0.9398" layer="1"/>
+<wire x1="44.831" y1="19.685" x2="44.45" y2="19.304" width="0.9398" layer="1"/>
+<wire x1="60.96" y1="17.887" x2="55.987" y2="22.86" width="0.9398" layer="1"/>
+<wire x1="55.987" y1="22.86" x2="44.831" y2="22.86" width="0.9398" layer="1"/>
 </signal>
 <signal name="N$3">
 <contactref element="C4" pad="2"/>
 <contactref element="POT1" pad="E"/>
-<wire x1="58.889" y1="46.99" x2="58.42" y2="38.0746" width="0" layer="19" extent="1-1"/>
+<wire x1="58.42" y1="38.0746" x2="58.42" y2="46.99" width="0.9398" layer="1"/>
+<wire x1="58.42" y1="46.99" x2="58.889" y2="46.99" width="0" layer="19" extent="1-1"/>
 </signal>
 <signal name="N$4">
@@
 <contactref element="T1" pad="2"/>
 <contactref element="C3" pad="1"/>
-<wire x1="24.13" y1="25.654" x2="13.97" y2="32.219" width="0" layer="19" extent="1-1"/>
-<wire x1="24.13" y1="41.656" x2="24.13" y2="25.654" width="0" layer="19" extent="1-1"/>
-<wire x1="37.592" y1="36.576" x2="24.13" y2="25.654" width="0" layer="19" extent="1-1"/>
+<wire x1="24.13" y1="25.654" x2="24.13" y2="33.02" width="0.9398" layer="1"/>
+<wire x1="24.13" y1="33.02" x2="24.13" y2="41.656" width="0.9398" layer="1"/>
+<wire x1="37.592" y1="32.766" x2="24.384" y2="32.766" width="0.9398" layer="1"/>
+<wire x1="24.384" y1="32.766" x2="24.13" y2="33.02" width="0.9398" layer="1"/>
+<wire x1="13.97" y1="33.489" x2="23.661" y2="33.489" width="0.9398" layer="1"/>
+<wire x1="23.661" y1="33.489" x2="24.13" y2="33.02" width="0.9398" layer="1"/>
 </signal>
 <signal name="N$5">
 <contactref element="R2" pad="P$2"/>
 <contactref element="C1" pad="1"/>
-<wire x1="24.13" y1="47.244" x2="12.7" y2="47.097" width="0" layer="19" extent="1-1"/>
+<wire x1="24.13" y1="47.244" x2="15.387" y2="47.244" width="0.9398" layer="1"/>
+<wire x1="15.387" y1="47.244" x2="12.7" y2="44.557" width="0.9398" layer="1"/>
 </signal>
 <signal name="N$6">
 <contactref element="R5" pad="P$2"/>
 <contactref element="R6" pad="P$1"/>
-<wire x1="28.194" y1="53.34" x2="39.116" y2="53.34" width="0" layer="19" extent="1-1"/>
+<wire x1="28.194" y1="53.34" x2="39.116" y2="53.34" width="0.9398" layer="1"/>
 </signal>
 <signal name="GND">
@@
 <contactref element="POT1" pad="A"/>
 <contactref element="R1" pad="P$1"/>
-<wire x1="12.7" y1="41.549" x2="58.42" y2="33.0454" width="0" layer="19" extent="1-1"/>
-<wire x1="24.13" y1="20.066" x2="12.7" y2="41.549" width="0" layer="19" extent="1-1"/>
-<wire x1="60.96" y1="12.339" x2="24.13" y2="20.066" width="0" layer="19" extent="1-1"/>
-<wire x1="45.72" y1="16.256" x2="60.96" y2="12.339" width="0" layer="19" extent="1-1"/>
 <polygon width="0.1524" layer="1">
 <vertex x="0" y="0"/>
@@
 <contactref element="H2" pad="PAD"/>
 <contactref element="C3" pad="2"/>
-<wire x1="13.97" y1="13.97" x2="13.97" y2="26.201" width="0" layer="19" extent="1-1"/>
+<wire x1="13.97" y1="27.471" x2="13.97" y2="13.97" width="0.9398" layer="1"/>
 </signal>
 <signal name="+12V">
 <contactref element="R6" pad="P$2"/>
 <contactref element="P+1" pad="VCC"/>
-<wire x1="11.43" y1="53.34" x2="22.606" y2="53.34" width="0" layer="19" extent="1-1"/>
+<wire x1="11.43" y1="53.34" x2="22.606" y2="53.34" width="0.9398" layer="1"/>
 </signal>
 <signal name="N$7">
 <contactref element="POT1" pad="S"/>
 <contactref element="H1" pad="PAD"/>
-<wire x1="71.12" y1="35.56" x2="60.96" y2="35.56" width="0" layer="19" extent="1-1"/>
+<wire x1="60.96" y1="35.56" x2="71.12" y2="35.56" width="0.9398" layer="1"/>
 </signal>
 </signals>
